Commit message: add tray holder xml

File: mujoco/g1_description/g1_tray_holder.urdf (robot description, URDF)
Before this commit: robot g1_29dof_with_hand_rev_1_0, 53 links, 52 joints
Links:
- removed link left_hand_index_0_link
- removed link left_hand_index_1_link
- removed link left_hand_middle_0_link
- removed link left_hand_middle_1_link
- removed link left_hand_palm_link
- removed link left_hand_thumb_0_link
- removed link left_hand_thumb_1_link
- removed link left_hand_thumb_2_link
- removed link right_hand_index_0_link
- removed link right_hand_index_1_link
- removed link right_hand_middle_0_link
- removed link right_hand_middle_1_link
- removed link right_hand_palm_link
- removed link right_hand_thumb_0_link
- removed link right_hand_thumb_1_link
- removed link right_hand_thumb_2_link
- added link left_tray_holder_link, mass 0.2; collision mesh filename=meshes/left_tray_holder_link_node__mesh_.obj scale=1. 1. 1.; visual mesh filename=meshes/left_tray_holder_link_node__mesh_.obj scale=1. 1. 1.
- added link right_tray_holder_link, mass 0.2; collision mesh filename=meshes/right_tray_holder_link_node__mesh_.obj scale=1. 1. 1.; visual mesh filename=meshes/right_tray_holder_link_node__mesh_.obj scale=1. 1. 1.
- added link world
Joints:
- removed joint left_hand_index_0_joint
- removed joint left_hand_index_1_joint
- removed joint left_hand_middle_0_joint
- removed joint left_hand_middle_1_joint
- removed joint left_hand_palm_joint
- removed joint left_hand_thumb_0_joint
- removed joint left_hand_thumb_1_joint
- removed joint left_hand_thumb_2_joint
- removed joint right_hand_index_0_joint
- removed joint right_hand_index_1_joint
- removed joint right_hand_middle_0_joint
- removed joint right_hand_middle_1_joint
- removed joint right_hand_palm_joint
- removed joint right_hand_thumb_0_joint
- removed joint right_hand_thumb_1_joint
- removed joint right_hand_thumb_2_joint
- added joint floating_base_joint: type floating, parent world, child pelvis
- added joint left_tray_holder_joint: type fixed, parent left_wrist_yaw_link, child left_tray_holder_link, origin xyz=0.0414958 -0.0000038 -0.0000005 rpy=-0.0000601 -0.0000552 0.0001914
- added joint right_tray_holder_joint: type fixed, parent right_wrist_yaw_link, child right_tray_holder_link, origin xyz=0.0414958 0.0000038 -0.0000005 rpy=0.0000601 -0.0000551 -0.0001914
